File: macropad3x3-kicad/macropad3x3.kicad_sch (KiCad schematic)
At the start: 0 parts

Commit message: schematic and pcb, matched outline to previous design
Parts:
- added D-BUTTON1, D-RE1, D-RE2, D1, D2, D3, D4, D5, D6, D7, D8, D9: Diode, Diode_THT:D_DO-41_SOD81_P10.16mm_Horizontal, symbol macropad:Diode-1N4148
- added J1: OLED-4PIN, macropad:OLED_128x32, symbol macropad:OLED-4PIN
- added MT1, MT2: Rotary-Enc-Switch, macropad:XDCR_PEC11R-4215F-S0024, symbol macropad:Rotary-Enc-Switch
- added S1, S2, S3, S4, S5, S6, S7, S8, S9: Keyswitch, macropad:MX_PCB_1.00u, symbol macropad:Keyswitch
- added S10: TS02-66-95-BK-260-LCR-D, macropad:SW_TS02-66-95-BK-260-LCR-D, symbol macropad:TS02-66-95-BK-260-LCR-D
- added U1: Arduino_Pro_Micro, macropad:Arduino_Pro_Micro, symbol macropad:MCU_Pro_Micro
Connections:
- new net: D2.2 (A), S2.2
- new net: D6.2 (A), S6.2
- new net: D5.2 (A), S5.2
- new net: D7.2 (A), S7.2
- new net: D8.2 (A), S8.2
- new net: D3.2 (A), S3.2
- new net: D4.2 (A), S4.2
- new net: D9.2 (A), S9.2
- new net: D1.2 (A), S1.2
- new net +5V: J1.VCC, U1.21 (VCC)
- new net Button1: S10.1, S2.1, S5.1, S8.1
- new net Button2: D-BUTTON1.2 (A), S10.3
- new net GND: J1.GND, MT1.COM, MT1.S1 (SHIELD), MT1.S2 (SHIELD), MT2.COM, MT2.S1 (SHIELD), MT2.S2 (SHIELD)
- new net RE1-1: MT1.1, S1.1, S4.1, S7.1
- new net RE1-2: D-RE1.2 (A), MT1.2
- new net RE2-1: MT2.1, S3.1, S6.1, S9.1
- new net RE2-2: D-RE2.2 (A), MT2.2
- new net SCL: J1.SCL
- new net SDA: J1.SDA
- new net row0: D-BUTTON1.1 (K), D-RE1.1 (K), D-RE2.1 (K)
- new net row1: D1.1 (K), D2.1 (K), D3.1 (K)
- new net row2: D4.1 (K), D5.1 (K), D6.1 (K)
- new net row3: D7.1 (K), D8.1 (K), D9.1 (K)

Commit message: hi
Parts:
- removed D-BUTTON1, D-RE1, D-RE2, D1, D2, D3, D4, D5, D6, D7, D8, D9: Diode, Diode_THT:D_DO-41_SOD81_P10.16mm_Horizontal, symbol macropad:Diode-1N4148
- removed J1: OLED-4PIN, macropad:OLED_128x32, symbol macropad:OLED-4PIN
- removed S10: TS02-66-95-BK-260-LCR-D, macropad:SW_TS02-66-95-BK-260-LCR-D, symbol macropad:TS02-66-95-BK-260-LCR-D
- added D-BUTTON1, D-RE1, D-RE2, D1, D2, D3, D4, D5, D6, D7, D8, D9: 1N4148, Diode_THT:D_DO-35_SOD27_P7.62mm_Horizontal, symbol Diode:1N4148
- added J1: OLED_128x32, macropad:OLED_128x32, symbol macropad:OLED_128x32
- added SW1: SW_Push_45deg, Button_Switch_THT:SW_PUSH_6mm, symbol Switch:SW_Push_45deg
Connections:
- net RE1-1 is gone; now on net col0: MT1.1, S1.1, S4.1, S7.1
- net RE2-2 is gone; now on net col2: MT2.2
- net Button1: now also U1.14 (16/PB2), SW1.1
- net Button2: now also D-BUTTON1.2 (A), SW1.2
- net RE1-2: now also D-RE1.2 (A)
- net RE2-1: now also D-RE2.2 (A); no longer S3.1, S6.1, S9.1
- net row0: now also D-BUTTON1.1 (K), D-RE1.1 (K), D-RE2.1 (K)
- net row1: now also D1.1 (K), D2.1 (K), D3.1 (K)
- net row2: now also D4.1 (K), D5.1 (K), D6.1 (K)
- net row3: now also D7.1 (K), D8.1 (K), D9.1 (K)
- net at S2.2: now also D2.2 (A)
- net at S6.2: now also D6.2 (A)
- net at S5.2: now also D5.2 (A)
- net at S7.2: now also D7.2 (A)
- net at S8.2: now also D8.2 (A)
- net at S3.2: now also D3.2 (A)
- net at S4.2: now also D4.2 (A)
- net at S9.2: now also D9.2 (A)
- net col2: now reaches U1.13 (10/PB6)
- net col2: now also S3.1, S6.1, S9.1
- net col0: now reaches U1.15 (14/PB3)
- net at S1.2: now also D1.2 (A)
- new net LED-DIN: U1.6 (3/PD0)
